File: Hardware/zk_48_ivg/zk_48_ivg.kicad_sch (KiCad schematic)
At the start: 26 parts, among them T1 IRF730

Commit message: Update
Parts:
- added C6: 22nF, symbol Device:C
- R1: value 100Ohm -> 100Ω
- R10, R9: value 100kOhm -> 100kΩ
- R11: value 270Ohm -> 270Ω
- R12: value 470Ohm -> 470Ω
- R13: value 670Ohm -> 670Ω
- R2, R3, R5: value 39kOhm -> 39kΩ
- R4, R6, R7: value 10kOhm -> 10kΩ
- R8: value 1kOhm -> 1kΩ
- renumbered C1 to U1, C2 to U2, C3 to U3
Connections:
- net +2V5: now also C6.1
- net GND: now also C6.2
