File: Hardware/zk_48_testrig/zk_48_testrig.kicad_sch (KiCad schematic)
At the start: 8 parts, among them T1 BC635

Commit message: Update
Parts:
- added J1: Port1, symbol Connector:Conn_01x02_Female
- added R1: 270Ω, symbol Device:R
- added R2: 15Ω, symbol Device:R
- added T1: BC635, Package_TO_SOT_THT:TO-92_Inline, symbol Transistor_BJT:BC337
Connections:
- net +15V: now also J1.1 (Pin_1)
- net GND: now also T1.3 (E)
- new net: R2.1, T1.1 (C)
- new net: R1.2, T1.2 (B)
- new net: J1.2 (Pin_2), R2.2
- new net FIRE: R1.1
Changed lines of the file:
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@@
+    (stroke (width 0) (type default) (color 0 0 0 0))
+  )
+  (wire (pts (xy 39.37 109.22) (xy 40.64 109.22))
     (stroke (width 0) (type default) (color 0 0 0 0))
   )
@@
     (stroke (width 0) (type default) (color 0 0 0 0))
   )
+  (wire (pts (xy 27.94 109.22) (xy 31.75 109.22))
+    (stroke (width 0) (type default) (color 0 0 0 0))
+  )
   (wire (pts (xy 24.13 67.31) (xy 24.13 57.15))
     (stroke (width 0) (type default) (color 0 0 0 0))
@@
     (stroke (width 0) (type default) (color 0 0 0 0))
   )
+  (wire (pts (xy 58.42 101.6) (xy 64.77 101.6))
+    (stroke (width 0) (type default) (color 0 0 0 0))
+  )
   (wire (pts (xy 66.04 21.59) (xy 66.04 26.67))
     (stroke (width 0) (type default) (color 0 0 0 0))
   )
+  (wire (pts (xy 62.23 96.52) (xy 62.23 99.06))
+    (stroke (width 0) (type default) (color 0 0 0 0))
+  )
   (wire (pts (xy 40.64 44.45) (xy 44.45 44.45))
     (stroke (width 0) (type default) (color 0 0 0 0))
@@
     (stroke (width 0) (type default) (color 0 0 0 0))
   )
+  (wire (pts (xy 48.26 104.14) (xy 48.26 101.6))
+    (stroke (width 0) (type default) (color 0 0 0 0))
+  )
   (wire (pts (xy 52.07 50.8) (xy 62.23 50.8))
     (stroke (width 0) (type default) (color 0 0 0 0))
@@
   )
   (wire (pts (xy 24.13 44.45) (xy 33.02 44.45))
+    (stroke (width 0) (type default) (color 0 0 0 0))
+  )
+  (wire (pts (xy 62.23 99.06) (xy 64.77 99.06))
+    (stroke (width 0) (type default) (color 0 0 0 0))
+  )
+  (wire (pts (xy 48.26 114.3) (xy 48.26 116.84))
+    (stroke (width 0) (type default) (color 0 0 0 0))
+  )
+  (wire (pts (xy 48.26 101.6) (xy 50.8 101.6))
     (stroke (width 0) (type default) (color 0 0 0 0))
   )
@@
     )
   )
+  (global_label "FIRE" (shape input) (at 27.94 109.22 180) (fields_autoplaced)
+    (effects (font (size 1.27 1.27)) (justify right))
+    (property "Intersheet References" "${INTERSHEET_REFS}" (id 0) (at 21.4145 109.1406 0)
+      (effects (font (size 1.27 1.27)) (justify right) hide)
+    )
+  )
   (symbol (lib_id "Device:R") (at 82.55 35.56 180) (unit 1)
     (in_bom yes) (on_board yes) (fields_autoplaced)
@@
     (pin "2")
   )
+  (symbol (lib_id "Transistor_BJT:BC337") (at 45.72 109.22 0) (unit 1)
+    (in_bom yes) (on_board yes) (fields_autoplaced)
+    (property "Reference" "T1" (id 0) (at 50.8 107.9499 0)
+      (effects (font (size 1.27 1.27)) (justify left))
+    )
+    (property "Value" "BC635" (id 1) (at 50.8 110.4899 0)
+      (effects (font (size 1.27 1.27)) (justify left))
+    )
+    (property "Footprint" "Package_TO_SOT_THT:TO-92_Inline" (id 2) (at 50.8 111.125 0)
+      (effects (font (size 1.27 1.27) italic) (justify left) hide)
+    )
+    (property "Datasheet" "https://diotec.com/tl_files/diotec/files/pdf/datasheets/bc337.pdf" (id 3) (at 45.72 109.22 0)
+      (effects (font (size 1.27 1.27)) (justify left) hide)
+    )
+    (pin "1")
+    (pin "2")
+    (pin "3")
+  )
   (symbol (lib_id "power:+15V") (at 66.04 21.59 0) (unit 1)
     (in_bom yes) (on_board yes) (fields_autoplaced)
@@
     (pin "1")
   )
+  (symbol (lib_id "power:+15V") (at 62.23 96.52 0) (unit 1)
+    (in_bom yes) (on_board yes) (fields_autoplaced)
+    (property "Reference" "#PWR?" (id 0) (at 62.23 100.33 0)
+      (effects (font (size 1.27 1.27)) hide)
+    )
+    (property "Value" "+15V" (id 1) (at 62.23 91.44 0))
+    (property "Footprint" "" (id 2) (at 62.23 96.52 0)
+      (effects (font (size 1.27 1.27)) hide)
+    )
+    (property "Datasheet" "" (id 3) (at 62.23 96.52 0)
+      (effects (font (size 1.27 1.27)) hide)
+    )
+    (pin "1")
+  )
   (symbol (lib_id "Device:R") (at 52.07 58.42 180) (unit 1)
     (in_bom yes) (on_board yes) (fields_autoplaced)
@@
     (pin "2")
   )
+  (symbol (lib_id "Connector:Conn_01x02_Female") (at 69.85 99.06 0) (unit 1)
+    (in_bom yes) (on_board yes) (fields_autoplaced)
+    (property "Reference" "J1" (id 0) (at 71.12 99.0599 0)
+      (effects (font (size 1.27 1.27)) (justify left))
+    )
+    (property "Value" "Port1" (id 1) (at 71.12 101.5999 0)
+      (effects (font (size 1.27 1.27)) (justify left))
+    )
+    (property "Footprint" "" (id 2) (at 69.85 99.06 0)
+      (effects (font (size 1.27 1.27)) hide)
+    )
+    (property "Datasheet" "~" (id 3) (at 69.85 99.06 0)
+      (effects (font (size 1.27 1.27)) hide)
+    )
+    (pin "1")
+    (pin "2")
+  )
+  (symbol (lib_id "Device:R") (at 54.61 101.6 90) (unit 1)
+    (in_bom yes) (on_board yes) (fields_autoplaced)
+    (property "Reference" "R2" (id 0) (at 54.61 95.25 90))
+    (property "Value" "15Ω" (id 1) (at 54.61 97.79 90))
+    (property "Footprint" "" (id 2) (at 54.61 103.378 90)
+      (effects (font (size 1.27 1.27)) hide)
+    )
+    (property "Datasheet" "~" (id 3) (at 54.61 101.6 0)
+      (effects (font (size 1.27 1.27)) hide)
+    )
+    (pin "1")
+    (pin "2")
+  )
   (symbol (lib_id "power:GND") (at 24.13 67.31 0) (unit 1)
     (in_bom yes) (on_board yes) (fields_autoplaced)
@@
     )
     (property "Datasheet" "" (id 3) (at 24.13 67.31 0)
+      (effects (font (size 1.27 1.27)) hide)
+    )
+    (pin "1")
+  )
+  (symbol (lib_id "power:GND") (at 48.26 116.84 0) (unit 1)
+    (in_bom yes) (on_board yes) (fields_autoplaced)
+    (property "Reference" "#PWR?" (id 0) (at 48.26 123.19 0)
+      (effects (font (size 1.27 1.27)) hide)
+    )
+    (property "Value" "GND" (id 1) (at 48.26 121.92 0))
+    (property "Footprint" "" (id 2) (at 48.26 116.84 0)
+      (effects (font (size 1.27 1.27)) hide)
+    )
+    (property "Datasheet" "" (id 3) (at 48.26 116.84 0)
       (effects (font (size 1.27 1.27)) hide)
     )
@@
     (pin "2")
     (pin "3")
+  )
+  (symbol (lib_id "Device:R") (at 35.56 109.22 90) (unit 1)
+    (in_bom yes) (on_board yes) (fields_autoplaced)
+    (property "Reference" "R1" (id 0) (at 35.56 102.87 90))
+    (property "Value" "270Ω" (id 1) (at 35.56 105.41 90))
+    (property "Footprint" "" (id 2) (at 35.56 110.998 90)
+      (effects (font (size 1.27 1.27)) hide)
+    )
+    (property "Datasheet" "~" (id 3) (at 35.56 109.22 0)
+      (effects (font (size 1.27 1.27)) hide)
+    )
+    (pin "1")
+    (pin "2")
   )
   (symbol (lib_id "Device:R") (at 58.42 36.83 90) (unit 1)
@@
       (reference "#PWR?") (unit 1) (value "+15V") (footprint "")
     )
+    (path "/3adb8c69-132c-478c-b246-f381b0e1424c"
+      (reference "#PWR?") (unit 1) (value "+15V") (footprint "")
+    )
     (path "/6ca7104b-aceb-41c7-9e01-e8c935c09261"
       (reference "#PWR?") (unit 1) (value "GND") (footprint "")
     )
+    (path "/713e4d09-6cf1-49fc-bf2e-c643eb7890b8"
+      (reference "#PWR?") (unit 1) (value "GND") (footprint "")
+    )
     (path "/9ace91c9-13a6-490f-bbff-869df4cd039c"
       (reference "#PWR?") (unit 1) (value "GND") (footprint "")
@@
       (reference "Bridge-Wire-Detonator") (unit 1) (value "4,7Ω") (footprint "")
     )
+    (path "/40ef82a7-1843-41e2-896c-620f16b91b4f"
+      (reference "J1") (unit 1) (value "Port1") (footprint "")
+    )
     (path "/d0d55c8b-16d6-4c3e-8041-1bc7d7f9e994"
       (reference "J?") (unit 1) (value "Module Connector") (footprint "")
@@
       (reference "J?") (unit 1) (value "Trigger Connector") (footprint "")
     )
+    (path "/b45301a2-b6d7-44bd-8834-616acde30aef"
+      (reference "R1") (unit 1) (value "270Ω") (footprint "")
+    )
     (path "/cc15f583-a41b-43af-ba94-a75455506a96"
       (reference "R1") (unit 1) (value "15Ω") (footprint "")
     )
+    (path "/6505825f-43ee-4fb8-b546-c0b2310ed040"
+      (reference "R2") (unit 1) (value "15Ω") (footprint "")
+    )
     (path "/79770cd5-32d7-429a-8248-0d9e6212231a"
       (reference "R2") (unit 1) (value "270Ω") (footprint "")
@@
       (reference "Shunt") (unit 1) (value "1Ω") (footprint "")
     )
+    (path "/09433d97-62ec-42de-89f2-7d0b68dc1b9d"
+      (reference "T1") (unit 1) (value "BC635") (footprint "Package_TO_SOT_THT:TO-92_Inline")
+    )
     (path "/9bac9ad3-a7b9-47f0-87c7-d8630653df68"
